File: Jitter_Cleaner.kicad_sch (KiCad schematic)
At the start: 44 parts, among them T1 TCM2-43X+, T3 TCM2-43X+, U18 SI5394, U20 TLV75733PDBV, U21 TLV75718PDBV, Y1 CX3225SB48000D0FPJC1

Commit message: Changes before submission
- Added pours to Jitter Cleaner0/VDD & Jitter Cleane1/VDD on In3 Layer
- Added knockout in planes on In2 layer under the XTAL shield
- Changed setback of ground layer from 0.5mm to 0.3mm
    - This fixed some breaks in the ground plane with dense vias, and cleared the way for uninterrupted gnd under controlled traces.
- Changed the 22uF 0805 XR7 16V cap to an instock 22uF 0805 XR7 25V
- Changed the 1uF 0603 XR7 16V cap to an instock 1uF 0603 XR7 25V
Parts:
- C137, C139, C141, C144: MPN GCM188R71C105KA64D -> GCM188R71E105KA64D
Changed lines of the file:
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@@
 			)
 		)
-		(property "Description" "CAP CER 1UF 16V X7R 0603"
+		(property "Description" "CAP CER 1UF 25V X7R 0603"
 			(at 285.75 88.9 0)
 			(effects
@@
 			)
 		)
-		(property "MPN" "GCM188R71C105KA64D"
+		(property "MPN" "GCM188R71E105KA64D"
 			(at 285.75 88.9 0)
 			(effects
@@
 			)
 		)
-		(property "Description" "CAP CER 1UF 16V X7R 0603"
+		(property "Description" "CAP CER 1UF 25V X7R 0603"
 			(at 269.24 105.41 0)
 			(effects
@@
 			)
 		)
-		(property "MPN" "GCM188R71C105KA64D"
+		(property "MPN" "GCM188R71E105KA64D"
 			(at 269.24 105.41 0)
 			(effects
@@
 			)
 		)
-		(property "Description" "CAP CER 1UF 16V X7R 0603"
+		(property "Description" "CAP CER 1UF 25V X7R 0603"
 			(at 193.04 106.68 0)
 			(effects
@@
 			)
 		)
-		(property "MPN" "GCM188R71C105KA64D"
+		(property "MPN" "GCM188R71E105KA64D"
 			(at 193.04 106.68 0)
 			(effects
@@
 			)
 		)
-		(property "Description" "CAP CER 1UF 16V X7R 0603"
+		(property "Description" "CAP CER 1UF 25V X7R 0603"
 			(at 184.15 88.9 0)
 			(effects
@@
 			)
 		)
-		(property "MPN" "GCM188R71C105KA64D"
+		(property "MPN" "GCM188R71E105KA64D"
 			(at 184.15 88.9 0)
 			(effects
