File: Power.kicad_sch (KiCad schematic)
At the start: 14 parts, among them U22 TPS563200

Commit message: Changes before submission
- Added pours to Jitter Cleaner0/VDD & Jitter Cleane1/VDD on In3 Layer
- Added knockout in planes on In2 layer under the XTAL shield
- Changed setback of ground layer from 0.5mm to 0.3mm
    - This fixed some breaks in the ground plane with dense vias, and cleared the way for uninterrupted gnd under controlled traces.
- Changed the 22uF 0805 XR7 16V cap to an instock 22uF 0805 XR7 25V
- Changed the 1uF 0603 XR7 16V cap to an instock 1uF 0603 XR7 25V
Parts:
- C136, C53, C54: MPN CL21A226MOCLRNC -> KGM21AR51E226MU; Manufacturer Samsung -> KYOCERA AVX
Changed lines of the file:
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@@
 			)
 		)
-		(property "Description" "CAP CER 22UF 16V X5R 0805"
+		(property "Description" "CAP CER 22UF 25V X5R 0805"
 			(at 179.07 88.9 0)
 			(effects
@@
 			)
 		)
-		(property "MPN" "CL21A226MOCLRNC"
+		(property "MPN" "KGM21AR51E226MU"
 			(at 179.07 88.9 0)
 			(effects
@@
 			)
 		)
-		(property "Manufacturer" "Samsung"
+		(property "Manufacturer" "KYOCERA AVX"
 			(at 179.07 88.9 0)
 			(effects
@@
 			)
 		)
-		(property "Description" "CAP CER 22UF 16V X5R 0805"
+		(property "Description" "CAP CER 22UF 25V X5R 0805"
 			(at 189.23 88.9 0)
 			(effects
@@
 			)
 		)
-		(property "MPN" "CL21A226MOCLRNC"
+		(property "MPN" "KGM21AR51E226MU"
 			(at 189.23 88.9 0)
 			(effects
@@
 			)
 		)
-		(property "Manufacturer" "Samsung"
+		(property "Manufacturer" "KYOCERA AVX"
 			(at 189.23 88.9 0)
 			(effects
@@
 			)
 		)
-		(property "Description" "CAP CER 22UF 16V X5R 0805"
+		(property "Description" "CAP CER 22UF 25V X5R 0805"
 			(at 214.63 88.9 0)
 			(effects
@@
 			)
 		)
-		(property "MPN" "CL21A226MOCLRNC"
+		(property "MPN" "KGM21AR51E226MU"
 			(at 214.63 88.9 0)
 			(effects
@@
 			)
 		)
-		(property "Manufacturer" "Samsung"
+		(property "Manufacturer" "KYOCERA AVX"
 			(at 214.63 88.9 0)
 			(effects
