File: eeprom.kicad_sch (KiCad schematic)
At the start: 9 parts, among them J19 WP Jumper, U9 AT24C64D

Commit message: Changes before submission
- Added pours to Jitter Cleaner0/VDD & Jitter Cleane1/VDD on In3 Layer
- Added knockout in planes on In2 layer under the XTAL shield
- Changed setback of ground layer from 0.5mm to 0.3mm
    - This fixed some breaks in the ground plane with dense vias, and cleared the way for uninterrupted gnd under controlled traces.
- Changed the 22uF 0805 XR7 16V cap to an instock 22uF 0805 XR7 25V
- Changed the 1uF 0603 XR7 16V cap to an instock 1uF 0603 XR7 25V
Parts:
- C33: MPN GCM188R71C105KA64D -> GCM188R71E105KA64D
Changed lines of the file:
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@@
 			)
 		)
-		(property "Description" "CAP CER 1UF 16V X7R 0603"
+		(property "Description" "CAP CER 1UF 25V X7R 0603"
 			(at 133.35 86.36 0)
 			(effects
@@
 			)
 		)
-		(property "MPN" "GCM188R71C105KA64D"
+		(property "MPN" "GCM188R71E105KA64D"
 			(at 133.35 86.36 0)
 			(effects
