File: fmc.kicad_sch (KiCad schematic)
At the start: 31 parts, among them P1 ASP-134488-01, Q1 FDN335N, Q2 FDN335N, Q3 FDN335N

Commit message: Changes before submission
- Added pours to Jitter Cleaner0/VDD & Jitter Cleane1/VDD on In3 Layer
- Added knockout in planes on In2 layer under the XTAL shield
- Changed setback of ground layer from 0.5mm to 0.3mm
    - This fixed some breaks in the ground plane with dense vias, and cleared the way for uninterrupted gnd under controlled traces.
- Changed the 22uF 0805 XR7 16V cap to an instock 22uF 0805 XR7 25V
- Changed the 1uF 0603 XR7 16V cap to an instock 1uF 0603 XR7 25V
Parts:
- C34, C35, C79: MPN CL21A226MOCLRNC -> KGM21AR51E226MU; Manufacturer Samsung -> KYOCERA AVX
Changed lines of the file:
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@@
 			)
 		)
-		(property "Description" "CAP CER 22UF 16V X5R 0805"
+		(property "Description" "CAP CER 22UF 25V X5R 0805"
 			(at 34.29 214.63 0)
 			(effects
@@
 			)
 		)
-		(property "MPN" "CL21A226MOCLRNC"
+		(property "MPN" "KGM21AR51E226MU"
 			(at 34.29 214.63 0)
 			(effects
@@
 			)
 		)
-		(property "Manufacturer" "Samsung"
+		(property "Manufacturer" "KYOCERA AVX"
 			(at 34.29 214.63 0)
 			(effects
@@
 			)
 		)
-		(property "Description" "CAP CER 22UF 16V X5R 0805"
+		(property "Description" "CAP CER 22UF 25V X5R 0805"
 			(at 34.29 189.23 0)
 			(effects
@@
 			)
 		)
-		(property "MPN" "CL21A226MOCLRNC"
+		(property "MPN" "KGM21AR51E226MU"
 			(at 34.29 189.23 0)
 			(effects
@@
 			)
 		)
-		(property "Manufacturer" "Samsung"
+		(property "Manufacturer" "KYOCERA AVX"
 			(at 34.29 189.23 0)
 			(effects
@@
 			)
 		)
-		(property "Description" "CAP CER 22UF 16V X5R 0805"
+		(property "Description" "CAP CER 22UF 25V X5R 0805"
 			(at 34.29 237.49 0)
 			(effects
@@
 			)
 		)
-		(property "MPN" "CL21A226MOCLRNC"
+		(property "MPN" "KGM21AR51E226MU"
 			(at 34.29 237.49 0)
 			(effects
@@
 			)
 		)
-		(property "Manufacturer" "Samsung"
+		(property "Manufacturer" "KYOCERA AVX"
 			(at 34.29 237.49 0)
 			(effects
