File: trigger-output-fmc.kicad_pcb (KiCad board)
At the start: 8 copper layers, 84 x 69 mm, 335 parts, among them J1 MMCX, J10 MMCX, J11 MMCX, J12 MMCX, J13 MMCX, J14 MMCX, J15 MMCX, J16 MMCX, J19 WP Jumper, J2 MMCX, J3 MMCX, J4 MMCX, J5 MMCX, J6 MMCX, J7 MMCX, J8 MMCX, J9 MMCX, P1 ASP-134488-01, Q1 FDN335N, Q2 FDN335N, Q3 FDN335N, T1 TCM2-43X+, T2 TCM2-43X+, T3 TCM2-43X+, T4 TCM2-43X+, U1 TLV3601, U10 SN74LVC2G126, U11 TLV3601, U12 SN74LVC2G126, U13 TLV3601, U14 SN74LVC2G126, U15 TLV3601, U16 SN74LVC2G126, U17 TLV3601, U18 SI5394, U19 SI5394, U2 TLV3601, U20 TLV75733PDBV, U21 TLV75718PDBV, U22 TPS563200, U23 74AVC4T245, U24 TLV75733PDBV, U25 74AVC4T245, U26 74LVC8T245, U27 74LVC8T245, U28 TLV75718PDBV, U29 SN74LVC2G126, U3 TLV3601, U30 TLV3601, U31 SN74LVC2G126, U32 TLV3601, U33 SN74LVC2G126, U34 TLV3601, U35 SN74LVC2G126, U36 TLV3601, U37 SN74LVC2G126, U38 TLV3601, U39 SN74LVC2G126, U4 SN74LVC2G126, U40 TLV3601, U41 SN74LVC2G126, U42 TLV3601, U43 SN74LVC2G126, U44 LP3855EMP-ADJ/NOPB, U48 SN74LVC2G126, U5 SN74LVC2G126, U6 TLV3601, U7 SN74LVC2G126, U8 TLV3601, U9 AT24C64D, Y1 CX3225SB48000D0FPJC1, Y2 CX3225SB48000D0FPJC1

Commit message: Changes before submission
- Added pours to Jitter Cleaner0/VDD & Jitter Cleane1/VDD on In3 Layer
- Added knockout in planes on In2 layer under the XTAL shield
- Changed setback of ground layer from 0.5mm to 0.3mm
    - This fixed some breaks in the ground plane with dense vias, and cleared the way for uninterrupted gnd under controlled traces.
- Changed the 22uF 0805 XR7 16V cap to an instock 22uF 0805 XR7 25V
- Changed the 1uF 0603 XR7 16V cap to an instock 1uF 0603 XR7 25V
Routing:
- added copper zone on In3.Cu, net /Jitter Cleaner0/VDD
- added copper zone on In3.Cu, net /Jitter Cleaner1/VDD
